File: smart_sensor_battery.kicad_pcb (KiCad board)
At the start: 2 copper layers, 23 x 56 mm, 30 parts, among them J1 Upper MCU Socket, J2 Lower MCU Socket, J3 Sensor Socket, J5 5-pin Socket, Q1 AO3401A, U2 BQ21040DBV, U4 TPS7A0533PDBV, U5 BQ29700, U6 CSD85301Q2, U7 SHTC3

Commit message: update to version 1.2
Parts:
- R10, R9: value 10k -> 3k3
- moved R10 31.4 mm to (128.0, 83.5), turned to 180 degrees
- turned R9 to 180 degrees
Connections:
- net BAT- renamed /BAT-
- net BATT_SENSE renamed /BAT_{SENSE}
- net MOSFET_DRAIN renamed /MOSFET_{DRAIN}
- net VUSB renamed /V_{USB}
- C2 pad 1: BAT+ -> /BAT+
- C3 pad 1: 3V3 -> +3V3
- C5 pad 1: 3V_SW -> /3V3_{SW}
- J1 pad 5: SDA -> /SDA
- J1 pad 6: SCL -> /SCL
- J2 pad 5: 3V3 -> +3V3
- J3 pad 1: 3V_SW -> /3V3_{SW}
- J3 pad 4: SCL -> /SCL
- J3 pad 5: SDA -> /SDA
- J5 pad 1: SDA -> /SDA
- J5 pad 2: SCL -> /SCL
- J5 pad 5: 3V_SW -> /3V3_{SW}
- Q1 pad 2: 3V3 -> +3V3
- Q1 pad 3: 3V_SW -> /3V3_{SW}
- R10 pad 1: SDA -> +3V3
- R10 pad 2: 3V_SW -> /SDA
- R12 pad 1: BAT+ -> /BAT+
- R4 pad 2: BAT+ -> /BAT+
- R7 pad 2: 3V3 -> +3V3
- R8 pad 2: BAT+ -> /BAT+
- R9 pad 1: SCL -> +3V3
- R9 pad 2: 3V_SW -> /SCL
- U2 pad 2: BAT+ -> /BAT+
- U4 pad 1: BAT+ -> /BAT+
- U4 pad 3: BAT+ -> /BAT+
- U4 pad 5: 3V3 -> +3V3
- U7 pad 1: 3V_SW -> /3V3_{SW}
- U7 pad 2: SCL -> /SCL
- U7 pad 3: SDA -> /SDA
Routing:
- net 3V_SW: track 100.9 -> 0.00 mm
- net /3V3_{SW}: track 0.00 -> 98.6 mm
- net SDA: track 88.7 -> 0.00 mm
- net /SDA: track 0.00 -> 80.2 mm
- net SCL: track 74.2 -> 0.00 mm, vias 2 -> 0
- net /SCL: track 0.00 -> 74.2 mm, vias 0 -> 2
- net +3V3: track 0.00 -> 45.1 mm
- net BAT+: track 38.1 -> 2.83 mm, vias 4 -> 0
- net /BAT+: track 0.00 -> 35.3 mm, vias 0 -> 4
- net 3V3: track 29.2 -> 0.00 mm
- net /BAT-: track 45.1 -> 44.3 mm
- net GND: vias 21 -> 22
- added copper zone on B.Cu, net /BAT+
- added copper zone on F.Cu, net /BAT+
- removed copper zone on B.Cu, net BAT+
- removed copper zone on F.Cu, net BAT+
Other:
- outline, holes or cut-outs redrawn
- board text added: "+"
- board text added: "-"
- board text added: "R. ${REVISION} ${ISSUE_DATE}"

Commit message: update to version 1.2b
Parts:
- added R13: 10k, Resistor_SMD:R_0402_1005Metric, F.Cu at (132.3, 100.7)
- added R14: 10k, Resistor_SMD:R_0402_1005Metric, F.Cu at (145.9, 57.7)
- added TP1: BAT+, TestPoint:TestPoint_Pad_4.0x4.0mm, B.Cu at (144.0, 58.0)
- added TP2: BAT-, TestPoint:TestPoint_Pad_4.0x4.0mm, B.Cu at (144.0, 109.0)
- moved R9 3.50 mm to (136.5, 100.2)
Connections:
- BT1 pad P: BAT+ -> /BAT+
- J3 pad 6: (no net) -> Net-(J1-Pin_2)
- J3 pad 7: (no net) -> Net-(J1-Pin_1)
Routing:
- net Net-(J1-Pin_2): track 0.00 -> 20.2 mm, vias 0 -> 2
- net Net-(J1-Pin_1): track 0.00 -> 20.1 mm, vias 0 -> 2
- net /BAT+: track 35.3 -> 46.0 mm
- net /BAT-: track 44.3 -> 54.1 mm
- net /SDA: track 80.2 -> 88.7 mm
- net +3V3: track 45.1 -> 41.6 mm
- net /SCL: track 74.2 -> 77.7 mm
- net BAT+: track 2.83 -> 0.00 mm
- net /3V3_{SW}: track 98.6 -> 100.1 mm
- net GND: vias 22 -> 21
