File: smart_sensor_battery.kicad_sch (KiCad schematic)
At the start: 11 parts, among them J1 Upper MCU Socket, J2 Lower MCU Socket, J3 Sensor Socket, J5 5-pin Socket, Q1 AO3401A, U1 XIAO-nRF52840, U7 SHTC3

Commit message: update to version 1.2
Parts:
- added BT1: 1096, CustomBattery:BAT_1096, symbol smart_sensor_battery:1096
- added C1, C2, C3: 2.2uF@16v, Capacitor_SMD:C_0603_1608Metric, symbol smart_sensor_battery:C
- added C4, C6: 100nF@16v, Capacitor_SMD:C_0402_1005Metric, symbol smart_sensor_battery:C
- added D1: LED, LED_SMD:LED_0402_1005Metric, symbol smart_sensor_battery:LED
- added R1: 1.2k, Resistor_SMD:R_0402_1005Metric, symbol smart_sensor_battery:R
- added R11, R12, R5, R6: 5.1M, Resistor_SMD:R_0402_1005Metric, symbol smart_sensor_battery:R
- added R2: 10k, Resistor_SMD:R_0402_1005Metric, symbol smart_sensor_battery:R
- added R3, R8: 2.2k, Resistor_SMD:R_0402_1005Metric, symbol smart_sensor_battery:R
- added R4: 330, Resistor_SMD:R_0402_1005Metric, symbol smart_sensor_battery:R
- added U2: BQ21040DBV, Package_TO_SOT_SMD:SOT-23-6, symbol smart_sensor_battery:BQ21040DBV
- added U4: TPS7A0533PDBV, Package_TO_SOT_SMD:SOT-23-5, symbol smart_sensor_battery:TPS7A0533PDBV
- added U5: BQ29700, Package_SON:WSON-6_1.5x1.5mm_P0.5mm, symbol smart_sensor_battery:BQ297xy
- added U6: CSD85301Q2, TI:CSD85301Q2, symbol smart_sensor_battery:CSD85301Q2_1
- J1, J2: symbol smart_sensor_battery:Conn_01x07_Socket -> Connector_Generic:Conn_01x07
- J3, J5: symbol smart_sensor_battery:Conn_01x05_Socket -> Connector_Generic:Conn_01x05
- R10, R9: value 10k -> 3k3; LCSC Part no. C25744 -> C60490
Connections:
- net GND: now also C1.2, C2.2, C3.2, C6.2, R1.2, R11.2, R2.2, R3.2, R5.2, U2.5 (GND), U4.2 (GND), U4.4 (NC_(GND)), U6.4 (S2)
- net SCL: now also R9.2; no longer R9.1
- net SDA: now also R10.2; no longer R10.1
- net 3V3 renamed +3V3
- net +3V3: now also R10.1, R9.1, C3.1, U4.5 (OUT)
- net 3V_SW renamed 3V3_{SW}
- net 3V3_{SW}: no longer R10.2, R9.2
- net BATT_SENSE renamed BAT_{SENSE}
- net BAT_{SENSE}: now also C6.1, R11.1, R12.2
- net VUSB renamed V_{USB}
- net V_{USB}: now also C1.1, U2.6 (VIN)
- new net: R5.1, U5.2 (Cout), U6.5 (G2)
- new net: R6.2, U5.3 (Dout), U6.2 (G1)
- new net: C4.1, R4.1, U5.5 (BAT)
- new net: R3.1, U5.6 (V-)
- new net: D1.1 (K), U2.3 (~{CHG})
- new net: D1.2 (A), R8.1
- new net: R2.1, U2.1 (TS)
- new net: R1.1, U2.4 (ISET)
- new net BAT+: BT1.P, C2.1, R12.1, R4.2, R8.2, U2.2 (OUT), U4.1 (IN), U4.3 (EN)
- new net BAT-: BT1.N, C4.2, R6.1, U5.4 (VSS), U6.1 (S1)
- new net MOSFET_{DRAIN}: U6.3 (D2), U6.6 (D1), U6.7 (D1), U6.8 (D2)
Other:
- removed sheet Battery Management
- note added: "Battery Charger IC"
- note added: "Battery Protection IC"
- note added: "Low Dropout Regulator (LDO)"
- moved on the sheet: C5, Q1, R10, R7, R9, U1, U7

Commit message: update to version 1.2b
Parts:
- added R13, R14: 10k, Resistor_SMD:R_0402_1005Metric, symbol smart_sensor_battery:R
- added TP1: BAT+, TestPoint:TestPoint_Pad_4.0x4.0mm, symbol Connector:TestPoint_Flag
- added TP2: BAT-, TestPoint:TestPoint_Pad_4.0x4.0mm, symbol Connector:TestPoint_Flag
- C1, C2, C3: LCSC (none) -> C23630; LCSC Part no. C23630 -> (none)
- C4, C5, C6: LCSC (none) -> C1525; LCSC Part no. C1525 -> (none)
- D1: LCSC (none) -> C74339; LCSC Part no. C74339 -> (none)
- J1, J2: LCSC (none) -> C42379199; LCSC Part no. C42379199 -> (none)
- J3: symbol Connector_Generic:Conn_01x05 -> Connector_Generic:Conn_01x07; LCSC (none) -> C42379199; LCSC Part no. C42379199 -> (none)
- J5: LCSC (none) -> C42379198; LCSC Part no. C42379198 -> (none)
- Q1: LCSC (none) -> C15127; LCSC Part no. C15127 -> (none)
- R1: LCSC (none) -> C25862; LCSC Part no. C25862 -> (none)
- R10, R9: LCSC (none) -> C60490; LCSC Part no. C60490 -> (none); now not fitted
- R11, R12, R5, R6: LCSC (none) -> C26092; LCSC Part no. C26092 -> (none)
- R2: LCSC (none) -> C25744; LCSC Part no. C25744 -> (none)
- R3, R8: LCSC (none) -> C25879; LCSC Part no. C25879 -> (none)
- R4: LCSC (none) -> C25104; LCSC Part no. C25104 -> (none)
- R7: LCSC (none) -> C25530; LCSC Part no. C25530 -> (none)
- U2: LCSC (none) -> C202311; LCSC Part no. C202311 -> (none)
- U4: LCSC (none) -> C493453; LCSC Part no. C493453 -> (none)
- U5: LCSC (none) -> C183096; LCSC Part no. C183096 -> (none)
- U6: LCSC (none) -> C544396; LCSC Part no. C544396 -> (none)
Connections:
- net 3V3_{SW}: now also R13.1, R14.1
- net BAT+: now also TP1.1
- net BAT-: now also TP2.1
- net SCL: now also R13.2
- net SDA: now also R14.2
- net at J1.1 (Pin_1), U1.1 (P0.02_A0_D0): now also J3.7 (Pin_7)
- net at J1.2 (Pin_2), U1.2 (P0.03_A1_D1): now also J3.6 (Pin_6)
Other:
- moved on the sheet: J5
